File: board/ParanoiaBox.kicad_pcb (KiCad board)
At the start: 2 copper layers, 68 x 89 mm, 60 parts, among them J1 Barrel_Jack, J2 RCAJack, J3 Conn_01x01, J4 Conn_01x01, J5 Conn_01x01, J6 Conn_01x01, J7 USB_B, J8 Conn_01x04, P1 Mini-DIN_6pins_ver4, Q1 2N2222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

Commit message: Changed TNTSChar.cpp to have less flicker, board to use wide transistors
Parts:
- Q1, Q2, Q3, Q4: footprint TO_SOT_Packages_THT:TO-92_Molded_Narrow -> TO_SOT_Packages_THT:TO-92_Inline_Wide
- moved Q1 5.25 mm to (120.6, 110.1)
- moved Q4 2.41 mm to (116.2, 96.5)
- moved Q3 1.89 mm to (129.7, 93.6)
- moved C18 1.65 mm to (129.8, 84.2)
- moved C13 1.48 mm to (134.4, 80.5)
- moved D1 1.32 mm to (121.0, 99.5)
- moved R11 0.98 mm to (114.0, 80.9)
- moved R8 0.89 mm to (121.6, 84.2)
- moved R10 0.81 mm to (123.8, 80.9)
- moved L1 0.72 mm to (114.3, 111.5)
- moved J2 0.31 mm to (117.7, 73.6)
- moved C7 0.25 mm to (119.9, 122.7)
Connections:
- J1 pad 3: (no net) -> Net-(J1-Pad3)
- P1 pad 2: (no net) -> Net-(P1-Pad2)
- P1 pad 6: (no net) -> Net-(P1-Pad6)
- Q3 pad 3: (no net) -> Net-(Q3-Pad3)
- Q4 pad 3: (no net) -> Net-(Q4-Pad3)
- U1 pad 9: (no net) -> Net-(U1-Pad9)
- U2 pad 9: (no net) -> Net-(U2-Pad9)
- UB1 pad 1: (no net) -> Net-(UB1-Pad1)
- UB1 pad 12: (no net) -> Net-(UB1-Pad12)
- UB1 pad 13: (no net) -> Net-(UB1-Pad13)
- UB1 pad 14: (no net) -> Net-(UB1-Pad14)
- UB1 pad 15: (no net) -> Net-(UB1-Pad15)
- UB1 pad 16: (no net) -> Net-(UB1-Pad16)
- UB1 pad 19: (no net) -> Net-(UB1-Pad19)
- UB1 pad 2: (no net) -> Net-(UB1-Pad2)
- UB1 pad 21: (no net) -> Net-(UB1-Pad21)
- UB1 pad 22: (no net) -> Net-(UB1-Pad22)
- UB1 pad 25: (no net) -> Net-(UB1-Pad25)
- UB1 pad 29: (no net) -> Net-(UB1-Pad29)
- UB1 pad 3: (no net) -> Net-(UB1-Pad3)
- UB1 pad 38: (no net) -> Net-(UB1-Pad38)
- UB1 pad 39: (no net) -> Net-(UB1-Pad39)
- UB1 pad 4: (no net) -> Net-(UB1-Pad4)
- UB1 pad 42: (no net) -> Net-(UB1-Pad42)
- UB1 pad 43: (no net) -> Net-(UB1-Pad43)
- UB1 pad 7: (no net) -> Net-(UB1-Pad7)
- UB1 pad 73: (no net) -> Net-(UB1-Pad73)
Routing:
- net Net-(Q1-Pad2): track 11.5 -> 6.05 mm
- net GND: track 654.9 -> 650.2 mm, vias 187 -> 183
- net +5V: track 390.5 -> 387.6 mm
- net Net-(Q2-Pad3): track 20.3 -> 17.6 mm
- net Net-(C14-Pad1): track 9.36 -> 6.75 mm
- net Net-(C12-Pad1): track 31.2 -> 28.9 mm
- net Net-(Q2-Pad2): track 19.4 -> 21.4 mm
- net Net-(C18-Pad2): track 15.7 -> 17.2 mm
- net +3V3: track 108.8 -> 110.3 mm
- net Net-(C14-Pad2): track 30.1 -> 29.2 mm
Other:
- board text added: "PARANOIABOX V2 BY D MARKS CC-BY-SA 4.0"
- board text removed: "PARANOIABOX BY D MARKS CC-BY-SA 4.0"
