File: board/ParanoiaBox.sch (KiCad schematic (older format))
At the start: 60 parts, among them J1 Barrel_Jack, J2 RCAJack, J3 Conn_01x01, J4 Conn_01x01, J5 Conn_01x01, J6 Conn_01x01, J7 USB_B, J8 Conn_01x04, P1 Mini-DIN_6pins_ver4, Q1 2N2222, Q2 2N3904, Q3 2N3904, Q4 2N3904, U1 MicroSD_SPI_CD, U2 MicroSD_SPI_CD, U3 NE555, U4 LM7805CT, U5 LM1117-3.3

Commit message: Changed TNTSChar.cpp to have less flicker, board to use wide transistors
Parts:
- Q1, Q2, Q3, Q4: footprint TO_SOT_Packages_THT:TO-92_Molded_Narrow -> TO_SOT_Packages_THT:TO-92_Inline_Wide
Changed lines of the file:
@@
 F 0 "Q1" H 5300 5675 50  0000 L CNN
 F 1 "2N2222" H 5300 5600 50  0000 L CNN
-F 2 "TO_SOT_Packages_THT:TO-92_Molded_Narrow" H 5300 5525 50  0001 L CIN
+F 2 "TO_SOT_Packages_THT:TO-92_Inline_Wide" H 5300 5525 50  0001 L CIN
 F 3 "" H 5100 5600 50  0001 L CNN
 	1    5100 5600
@@
 F 0 "Q2" H 3300 5925 50  0000 L CNN
 F 1 "2N3904" H 3300 5850 50  0000 L CNN
-F 2 "TO_SOT_Packages_THT:TO-92_Molded_Narrow" H 3300 5775 50  0001 L CIN
+F 2 "TO_SOT_Packages_THT:TO-92_Inline_Wide" H 3300 5775 50  0001 L CIN
 F 3 "" H 3100 5850 50  0001 L CNN
 	1    3100 5850
@@
 F 0 "Q3" H 6450 5275 50  0000 L CNN
 F 1 "2N3904" H 6450 5200 50  0000 L CNN
-F 2 "TO_SOT_Packages_THT:TO-92_Molded_Narrow" H 6450 5125 50  0001 L CIN
+F 2 "TO_SOT_Packages_THT:TO-92_Inline_Wide" H 6450 5125 50  0001 L CIN
 F 3 "" H 6250 5200 50  0001 L CNN
 	1    6250 5200
@@
 F 0 "Q4" H 8400 5175 50  0000 L CNN
 F 1 "2N3904" H 8400 5100 50  0000 L CNN
-F 2 "TO_SOT_Packages_THT:TO-92_Molded_Narrow" H 8400 5025 50  0001 L CIN
+F 2 "TO_SOT_Packages_THT:TO-92_Inline_Wide" H 8400 5025 50  0001 L CIN
 F 3 "" H 8200 5100 50  0001 L CNN
 	1    8200 5100
